File: pcb/snappy.kicad_pcb (KiCad board)
At the start: 4 copper layers, 10.2 x 25.4 mm, 22 parts, among them J1 Conn_01x04_Male, J2 Conn_01x04_Male, J3 Conn_01x03_Male, J4 Conn_01x03_Male, J5 Conn_01x03_Male, J6 Conn_01x03_Male, U1 ATtiny3216-M

Commit message: Add files via upload
Parts:
- removed G***: LOGO, mothface:mothfacesmolest
